File: Hardware/LEDBadge.sch (KiCad schematic (older format))
At the start: 27 parts

Commit message: Update
Parts:
- added BT1: CR2032, Hardware:CCR-2008, symbol Battery_Cell
- added C1, C2: 10uF, Capacitors_SMD:C_0805, symbol C
- BT2: renamed from BT?; value Battery_Cell -> CR2032; footprint (none) -> Hardware:CCR-2008
- D1, D10, D11, D12, D13, D14, D15, D16, D2, D3, D4, D5, D6, D7, D8, D9: renamed from D?; footprint (none) -> LEDs:LED_0603
- J1: renamed from J?; footprint (none) -> Pin_Headers:Pin_Header_Straight_2x03_Pitch2.54mm
- R1: renamed from R?; value 10K -> 1K; footprint (none) -> Resistors_SMD:R_0603
- R2: renamed from R?; footprint (none) -> Resistors_SMD:R_0603
- R3, R4, R5, R6: renamed from R?; value R -> 180; footprint (none) -> Resistors_SMD:R_0603
- SW1: renamed from SW?; footprint (none) -> Buttons_Switches_SMD:SW_SPST_SKQG
- U1: renamed from U?; footprint TQFP32 -> Housings_QFP:TQFP-32_7x7mm_Pitch0.8mm
- U2: renamed from U?; footprint (none) -> Hardware:NRF24L01-SMD
Connections:
- net +BATT: now also BT1.1 (+), C1.1, C2.1
- net GND: now also BT1.2 (-), C1.2, C2.2
Other:
- moved on the sheet: R2, U2
